File: clockPCB/clockPCB.kicad_pcb (KiCad board)
At the start: 2 copper layers, 27.7 x 142.5 mm, 13 parts

Commit message: pcb
Parts:
- added ?: , , F.Cu at (148.8, 97.0)
- added ?: , , F.Cu at (148.8, 83.2)
- added ?: , , F.Cu at (148.8, 75.6)
- added ?: , , F.Cu at (148.8, 131.0)
- added ?: , , F.Cu at (148.8, 107.1)
- added ?: , , F.Cu at (148.8, 78.2)
- added ?: , , F.Cu at (148.8, 123.4)
- added ?: , , F.Cu at (148.8, 115.8)
- added ?: , , F.Cu at (148.8, 73.1)
- added ?: , , F.Cu at (148.8, 91.9)
- added ?: , , F.Cu at (148.8, 68.0)
- added ?: , , F.Cu at (148.8, 120.8)
- added ?: , , F.Cu at (148.8, 125.9)
- added ?: , , F.Cu at (148.8, 85.8)
- added ?: , , F.Cu at (148.8, 102.0)
- added REF**: 0.1uF Ceramic, Luminator:0.1uF Ceramic, F.Cu at (125.0, 67.5)
- added REF**: 2.25x1.5 PAD, Luminator:2.25x1.5 PAD, F.Cu at (148.8, 128.5)
- added REF**: 2.25x1.5 PAD, Luminator:2.25x1.5 PAD, F.Cu at (148.8, 109.7)
- added REF**: 2.25x1.5 PAD, Luminator:2.25x1.5 PAD, F.Cu at (148.8, 99.5)
- added REF**: 2.25x1.5 PAD, Luminator:2.25x1.5 PAD, F.Cu at (148.8, 104.6)
- added REF**: 2.25x1.5 PAD, Luminator:2.25x1.5 PAD, F.Cu at (148.8, 133.5)
- added REF**: CP_Radial_D5.0mm_P2.50mm, Capacitor_THT:CP_Radial_D5.0mm_P2.50mm, F.Cu at (148.8, 150.0)
- added REF**: 0.1uF Ceramic, Luminator:0.1uF Ceramic, F.Cu at (125.7, 139.6)
- added REF**: 2.25x1.5 PAD, Luminator:2.25x1.5 PAD, F.Cu at (148.8, 70.5)
- added REF**: 2.25x1.5 PAD, Luminator:2.25x1.5 PAD, F.Cu at (148.8, 94.4)
- added REF**: 2.25x6.1 PAD_1, Luminator:2.25x6.1 PAD_1, F.Cu at (148.8, 141.7)
- added REF**: 2.25x1.5 PAD, Luminator:2.25x1.5 PAD, F.Cu at (148.8, 118.3)
- added REF**: 2.25x1.5 PAD, Luminator:2.25x1.5 PAD, F.Cu at (148.8, 80.7)
- moved REF** 6.31 mm to (129.6, 117.3)
- moved REF** 6.31 mm to (136.1, 91.9)
- moved REF** 6.31 mm to (129.6, 69.6)
- moved REF** 6.31 mm to (135.6, 41.3)
- moved REF** 6.31 mm to (138.9, 91.9)
- moved REF** 6.31 mm to (136.1, 68.0)
- moved REF** 6.31 mm to (138.9, 68.0)
- moved REF** 6.31 mm to (129.7, 146.5)
- moved REF** 6.31 mm to (136.1, 115.8)
- moved REF** 6.31 mm to (129.6, 93.5)
- moved REF** 6.31 mm to (139.3, 146.9)
- moved REF** 6.31 mm to (138.9, 115.8)
- moved REF** 5.83 mm to (135.9, 156.1)
Routing:
- net (no net): track 1492.7 -> 1859.2 mm, vias 14 -> 16
Other:
- board size 27.7 x 142.5 mm -> 28.2 x 142.5 mm
- board text added: "12v -> 5v PXO78-500-M"
- board text added: "FlipDot Clock Crontroller (rev 1.0), Designed by Tyler Bowers 2023, Idea by Elizabeth Johnson"
- board text added: "GND"
- board text added: "RTC"
- board text added: "SN74AHC595"

Commit message: asd
Routing:
- net (no net): track 1859.2 -> 1930.7 mm
Other:
- board text added: "^ USB"

Commit message: asd
Routing:
- net (no net): track 1930.7 -> 1904.6 mm
Changed lines of the file:
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@@
   (segment (start 129.6035 87.0585) (end 134.874 87.0585) (width 0.25) (layer "F.Cu") (net 0))
   (segment (start 133.4135 104.5845) (end 131.318 104.5845) (width 0.25) (layer "F.Cu") (net 0))
-  (segment (start 147.066 36.2585) (end 131.826 36.2585) (width 0.2) (layer "F.Cu") (net 0))
   (segment (start 128.27 138.6205) (end 128.27 139.5965) (width 0.2) (layer "F.Cu") (net 0))
   (segment (start 143.51 27.1145) (end 147.066 23.5585) (width 0.2) (layer "F.Cu") (net 0))
@@
   (segment (start 129.6035 76.8985) (end 134.874 76.8985) (width 0.25) (layer "F.Cu") (net 0))
   (segment (start 146.05 66.2305) (end 147.574 66.2305) (width 0.2) (layer "F.Cu") (net 0))
-  (segment (start 131.826 36.2585) (end 124.206 43.8785) (width 0.2) (layer "F.Cu") (net 0))
   (segment (start 139.446 156.6545) (end 143.932 152.1685) (width 0.2) (layer "F.Cu") (net 0))
   (segment (start 131.6355 92.6465) (end 123.952 92.6465) (width 0.25) (layer "F.Cu") (net 0))

Commit message: asd
Routing:
- net (no net): track 1904.6 -> 1933.3 mm
Changed lines of the file:
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@@
   (segment (start 134.874 81.9785) (end 136.144 80.7085) (width 0.25) (layer "F.Cu") (net 0))
   (segment (start 129.6035 105.8545) (end 134.874 105.8545) (width 0.25) (layer "F.Cu") (net 0))
-  (segment (start 140.208 112.2045) (end 140.208 88.3285) (width 0.4) (layer "F.Cu") (net 0))
   (segment (start 134.874 129.7305) (end 136.144 128.4605) (width 0.25) (layer "F.Cu") (net 0))
   (segment (start 123.952 116.5225) (end 123.952 134.0485) (width 0.25) (layer "F.Cu") (net 0))
@@
   (segment (start 144.526 148.2725) (end 144.526 141.6685) (width 0.2) (layer "F.Cu") (net 0))
   (segment (start 136.144 78.1685) (end 138.684 75.6285) (width 0.25) (layer "F.Cu") (net 0))
+  (segment (start 140.208 67.31) (end 140.208 89.154) (width 0.25) (layer "F.Cu") (net 0))
   (segment (start 127 69.2785) (end 127.488 68.7905) (width 0.2) (layer "F.Cu") (net 0))
   (segment (start 125.7935 70.5485) (end 129.6035 74.3585) (width 0.25) (layer "F.Cu") (net 0))
@@
   (segment (start 134.874 103.3145) (end 136.144 102.0445) (width 0.25) (layer "F.Cu") (net 0))
   (segment (start 125.7935 123.3805) (end 129.6035 127.1905) (width 0.25) (layer "F.Cu") (net 0))
+  (segment (start 137.3505 90.678) (end 140.208 90.678) (width 0.25) (layer "F.Cu") (net 0))
   (segment (start 125.7935 120.8405) (end 129.6035 124.6505) (width 0.25) (layer "F.Cu") (net 0))
   (segment (start 133.4135 70.5485) (end 128.27 70.5485) (width 0.25) (layer "F.Cu") (net 0))
@@
   (segment (start 123.952 116.5225) (end 123.952 92.6465) (width 0.25) (layer "F.Cu") (net 0))
   (segment (start 148.844 83.2485) (end 146.558 83.2485) (width 0.25) (layer "F.Cu") (net 0))
+  (segment (start 137.3505 114.554) (end 140.208 114.554) (width 0.25) (layer "F.Cu") (net 0))
   (segment (start 136.144 112.2045) (end 138.684 109.6645) (width 0.25) (layer "F.Cu") (net 0))
   (segment (start 148.844 68.0085) (end 146.558 68.0085) (width 0.25) (layer "F.Cu") (net 0))
@@
   (segment (start 136.144 90.1065) (end 135.5725 90.678) (width 0.25) (layer "F.Cu") (net 0))
   (segment (start 135.9535 118.3005) (end 136.144 118.3005) (width 0.25) (layer "F.Cu") (net 0))
-  (segment (start 140.208 136.0805) (end 140.208 112.2045) (width 0.4) (layer "F.Cu") (net 0))
   (segment (start 148.844 85.7885) (end 146.558 85.7885) (width 0.25) (layer "F.Cu") (net 0))
   (segment (start 125.7935 102.0445) (end 129.6035 105.8545) (width 0.25) (layer "F.Cu") (net 0))
@@
   (segment (start 141.986 156.6545) (end 144.272 154.3685) (width 0.2) (layer "F.Cu") (net 0))
   (segment (start 136.144 73.0885) (end 138.684 70.5485) (width 0.25) (layer "F.Cu") (net 0))
+  (segment (start 140.208 90.678) (end 140.208 89.154) (width 0.4) (layer "F.Cu") (net 0))
   (segment (start 135.5725 90.678) (end 129.3495 90.678) (width 0.25) (layer "F.Cu") (net 0))
   (segment (start 126.492 138.6205) (end 128.27 138.6205) (width 0.2) (layer "F.Cu") (net 0))
@@
   (segment (start 138.684 125.9205) (end 138.938 125.9205) (width 0.25) (layer "F.Cu") (net 0))
   (segment (start 138.684 109.6645) (end 138.938 109.6645) (width 0.25) (layer "F.Cu") (net 0))
-  (segment (start 133.4135 70.5485) (end 135.9535 68.0085) (width 0.25) (layer "F.Cu") (net 0))
   (segment (start 148.844 128.4605) (end 146.558 128.4605) (width 0.25) (layer "F.Cu") (net 0))
   (segment (start 125.7935 118.3005) (end 129.6035 122.1105) (width 0.25) (layer "F.Cu") (net 0))
   (segment (start 133.25475 83.2485) (end 130.556 83.2485) (width 0.25) (layer "F.Cu") (net 0))
+  (segment (start 140.208 136.0805) (end 140.208 114.554) (width 0.4) (layer "F.Cu") (net 0))
   (segment (start 129.88925 85.7885) (end 129.794 85.7885) (width 0.25) (layer "F.Cu") (net 0))
   (segment (start 129.88925 85.7885) (end 129.88925 85.7885) (width 0.25) (layer "F.Cu") (net 0))
@@
   (segment (start 147.066 36.2585) (end 149.098 38.2905) (width 0.2) (layer "F.Cu") (net 0))
   (segment (start 134.874 105.8545) (end 136.144 104.5845) (width 0.25) (layer "F.Cu") (net 0))
+  (segment (start 140.208 112.2045) (end 140.208 90.678) (width 0.4) (layer "F.Cu") (net 0))
   (segment (start 142.494 57.5945) (end 138.938 54.0385) (width 0.25) (layer "F.Cu") (net 0))
   (segment (start 148.844 125.9205) (end 146.558 125.9205) (width 0.25) (layer "F.Cu") (net 0))
@@
   (segment (start 136.144 131.0005) (end 138.684 128.4605) (width 0.25) (layer "F.Cu") (net 0))
   (segment (start 148.844 104.5845) (end 146.558 104.5845) (width 0.25) (layer "F.Cu") (net 0))
+  (segment (start 136.144 115.7605) (end 137.3505 114.554) (width 0.25) (layer "F.Cu") (net 0))
   (segment (start 138.684 115.7605) (end 138.938 115.7605) (width 0.25) (layer "F.Cu") (net 0))
   (segment (start 129.794 85.7885) (end 129.794 85.69325) (width 0.25) (layer "F.Cu") (net 0))
   (segment (start 129.6035 87.0585) (end 134.874 87.0585) (width 0.25) (layer "F.Cu") (net 0))
   (segment (start 133.4135 104.5845) (end 131.318 104.5845) (width 0.25) (layer "F.Cu") (net 0))
+  (segment (start 140.208 114.554) (end 140.208 112.2045) (width 0.4) (layer "F.Cu") (net 0))
   (segment (start 128.27 138.6205) (end 128.27 139.5965) (width 0.2) (layer "F.Cu") (net 0))
+  (segment (start 137.3505 66.802) (end 139.7 66.802) (width 0.25) (layer "F.Cu") (net 0))
   (segment (start 143.51 27.1145) (end 147.066 23.5585) (width 0.2) (layer "F.Cu") (net 0))
   (segment (start 133.4135 120.8405) (end 135.9535 118.3005) (width 0.25) (layer "F.Cu") (net 0))
@@
   (segment (start 136.144 88.3285) (end 138.684 85.7885) (width 0.25) (layer "F.Cu") (net 0))
   (segment (start 143.932 152.1685) (end 144.526 152.1685) (width 0.2) (layer "F.Cu") (net 0))
-  (segment (start 133.4135 118.3005) (end 135.9535 115.7605) (width 0.25) (layer "F.Cu") (net 0))
   (segment (start 149.098 28.1305) (end 147.066 26.0985) (width 0.2) (layer "F.Cu") (net 0))
   (segment (start 129.698 145.9965) (end 129.698 146.4945) (width 0.4) (layer "F.Cu") (net 0))
   (segment (start 138.684 85.7885) (end 138.938 85.7885) (width 0.25) (layer "F.Cu") (net 0))
   (segment (start 146.05 154.3685) (end 146.304 154.1145) (width 0.2) (layer "F.Cu") (net 0))
+  (segment (start 139.7 66.802) (end 140.208 67.31) (width 0.25) (layer "F.Cu") (net 0))
   (segment (start 141.478 57.8485) (end 140.208 56.5785) (width 0.25) (layer "F.Cu") (net 0))
   (segment (start 148.844 107.1245) (end 146.558 107.1245) (width 0.25) (layer "F.Cu") (net 0))
@@
   (segment (start 138.684 118.3005) (end 138.938 118.3005) (width 0.25) (layer "F.Cu") (net 0))
   (segment (start 148.844 147.5105) (end 148.844 141.6685) (width 0.4) (layer "F.Cu") (net 0))
+  (segment (start 140.208 89.154) (end 140.208 88.3285) (width 0.4) (layer "F.Cu") (net 0))
   (segment (start 123.952 134.0485) (end 123.952 136.0805) (width 0.2) (layer "F.Cu") (net 0))
   (segment (start 140.208 112.2045) (end 138.938 112.2045) (width 0.4) (layer "F.Cu") (net 0))
@@
   (segment (start 134.874 122.1105) (end 136.144 120.8405) (width 0.25) (layer "F.Cu") (net 0))
   (segment (start 144.272 154.3685) (end 146.05 154.3685) (width 0.2) (layer "F.Cu") (net 0))
+  (segment (start 136.144 68.0085) (end 137.3505 66.802) (width 0.25) (layer "F.Cu") (net 0))
   (segment (start 129.6035 127.1905) (end 134.874 127.1905) (width 0.25) (layer "F.Cu") (net 0))
   (segment (start 129.6035 124.6505) (end 134.874 124.6505) (width 0.25) (layer "F.Cu") (net 0))
@@
   (segment (start 129.6035 103.3145) (end 134.874 103.3145) (width 0.25) (layer "F.Cu") (net 0))
   (segment (start 143.002 150.6445) (end 144.526 152.1685) (width 0.2) (layer "F.Cu") (net 0))
-  (segment (start 133.4135 94.4245) (end 135.9535 91.8845) (width 0.25) (layer "F.Cu") (net 0))
   (segment (start 129.6035 129.7305) (end 134.874 129.7305) (width 0.25) (layer "F.Cu") (net 0))
   (segment (start 134.874 137.3505) (end 136.144 136.0805) (width 0.25) (layer "F.Cu") (net 0))
@@
   (segment (start 131.6355 92.6465) (end 123.952 92.6465) (width 0.25) (layer "F.Cu") (net 0))
   (segment (start 148.844 102.0445) (end 146.558 102.0445) (width 0.25) (layer "F.Cu") (net 0))
+  (segment (start 136.144 91.8845) (end 137.3505 90.678) (width 0.25) (layer "F.Cu") (net 0))
   (segment (start 135.9535 68.0085) (end 136.144 68.0085) (width 0.25) (layer "F.Cu") (net 0))
   (segment (start 123.952 70.0405) (end 123.952 92.6465) (width 0.25) (layer "F.Cu") (net 0))
@@
   (segment (start 124.206 43.8785) (end 122.682 45.4025) (width 0.2) (layer "B.Cu") (net 0))
   (segment (start 148.844 153.0985) (end 148.844 150.0105) (width 0.4) (layer "B.Cu") (net 0))
-  (segment (start 136.144 68.0085) (end 136.144 34.4805) (width 0.25) (layer "B.Cu") (net 0))
   (segment (start 131.318 126.365) (end 131.318 104.5845) (width 0.25) (layer "B.Cu") (net 0))
   (segment (start 124.206 38.7985) (end 130.556 45.1485) (width 0.25) (layer "B.Cu") (net 0))
@@
   (segment (start 130.556 79.9465) (end 131.318 80.7085) (width 0.25) (layer "B.Cu") (net 0))
   (segment (start 131.318 77.4065) (end 131.318 43.3705) (width 0.25) (layer "B.Cu") (net 0))
+  (segment (start 133.4135 37.211) (end 147.066 23.5585) (width 0.25) (layer "B.Cu") (net 0))
   (segment (start 129.032 56.3245) (end 129.032 85.0265) (width 0.25) (layer "B.Cu") (net 0))
-  (segment (start 136.144 34.4805) (end 147.066 23.5585) (width 0.25) (layer "B.Cu") (net 0))
   (segment (start 141.986 139.1285) (end 142.24 139.1285) (width 0.2) (layer "B.Cu") (net 0))
   (segment (start 130.556 83.2485) (end 129.794 82.4865) (width 0.25) (layer "B.Cu") (net 0))
@@
   (segment (start 145.034 112.2045) (end 145.034 136.0805) (width 0.25) (layer "B.Cu") (net 0))
   (segment (start 132.08 74.295) (end 133.4135 75.6285) (width 0.25) (layer "B.Cu") (net 0))
+  (segment (start 133.4135 70.5485) (end 133.4135 37.211) (width 0.25) (layer "B.Cu") (net 0))
 )

Commit message: asd
Parts:
- removed the REF** at (138.9, 115.8)
- removed the REF** at (138.9, 91.9)
- removed the REF** at (138.9, 68.0)
- added REF**: TBD62783APG, Luminator:TBD62783APG, F.Cu at (138.9, 91.9)
- added REF**: TBD62783APG, Luminator:TBD62783APG, F.Cu at (138.9, 115.8)
- added REF**: TBD62783APG, Luminator:TBD62783APG, F.Cu at (138.9, 68.1)
Routing:
- net (no net): track 1933.3 -> 1932.1 mm

Commit message: asd
Routing:
- net (no net): track 1932.1 -> 1978.5 mm
Changed lines of the file:
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@@
   (segment (start 124.46 68.0285) (end 124.988 67.5005) (width 0.2) (layer "B.Cu") (net 0))
   (segment (start 122.682 27.6225) (end 124.206 26.0985) (width 0.2) (layer "B.Cu") (net 0))
+  (segment (start 136.144 37.0205) (end 147.066 26.0985) (width 0.25) (layer "B.Cu") (net 0))
   (segment (start 129.698 152.9405) (end 127.762 154.8765) (width 0.4) (layer "B.Cu") (net 0))
   (segment (start 129.794 46.9265) (end 124.206 41.3385) (width 0.25) (layer "B.Cu") (net 0))
+  (segment (start 136.144 68.0085) (end 136.144 37.0205) (width 0.25) (layer "B.Cu") (net 0))
   (segment (start 125.7935 88.3285) (end 124.46 89.662) (width 0.25) (layer "B.Cu") (net 0))
   (segment (start 132.08 102.0445) (end 132.08 124.587) (width 0.25) (layer "B.Cu") (net 0))

Commit message: Public release update
Other:
- board text added: "You can also use TBD62783APG, or TBD62786APG for the transistor array. The difference is that the TBD62786APG is output low when input high, and output high when input low. TBD62783APG is output low when input low, and output high when input high. Please make sure that the board is configured correctly for using the chip you choose."
Changed lines of the file:
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@@
+    (effects (font (size 1.5 1.5) (thickness 0.3) bold) (justify left bottom))
+  )
+  (gr_text "You can also use TBD62783APG, or TBD62786APG for the transistor array.\nThe difference is that the TBD62786APG is output low when input high, and output high when input low.\nTBD62783APG is output low when input low, and output high when input high.\nPlease make sure that the board is configured correctly for using the chip you choose.\n" (at 155.5496 84.8614) (layer "Cmts.User")
     (effects (font (size 1.5 1.5) (thickness 0.3) bold) (justify left bottom))
   )
